Commit message: Updated the xacro generated reemc model urdf
git-svn-id: svn+ssh://server/srv/svn/repos/trunk/pal-ros-pkg/catkin_pkgs/reemc_simulation@52391 5e370ff8-3418-0410-babe-3378cc20a00d

File: reemc_gazebo/models/reemc_full/model.urdf (robot description, URDF)
Before this commit: robot reemc, 71 links, 70 joints
Joints:
- joint hand_left_index_1_joint: mimic joint=hand_left_index_joint multiplier=-1.0 offset=0.0 -> joint=hand_left_index_joint multiplier=0.36 offset=0.0
- joint hand_left_index_2_joint: mimic joint=hand_left_index_joint multiplier=-1.0 offset=0.0 -> joint=hand_left_index_joint multiplier=0.32 offset=0.0
- joint hand_left_index_3_joint: mimic joint=hand_left_index_joint multiplier=-1.0 offset=0.0 -> joint=hand_left_index_joint multiplier=0.32 offset=0.0
- joint hand_left_middle_1_joint: mimic joint=hand_left_middle_joint multiplier=-1.0 offset=0.0 -> joint=hand_left_middle_joint multiplier=0.36 offset=0.0
- joint hand_left_middle_2_joint: mimic joint=hand_left_middle_joint multiplier=-1.0 offset=0.0 -> joint=hand_left_middle_joint multiplier=0.32 offset=0.0
- joint hand_left_middle_3_joint: mimic joint=hand_left_middle_joint multiplier=-1.0 offset=0.0 -> joint=hand_left_middle_joint multiplier=0.32 offset=0.0
- joint hand_right_index_1_joint: mimic joint=hand_right_index_joint multiplier=-1.0 offset=0.0 -> joint=hand_right_index_joint multiplier=0.36 offset=0.0
- joint hand_right_index_2_joint: mimic joint=hand_right_index_joint multiplier=-1.0 offset=0.0 -> joint=hand_right_index_joint multiplier=0.32 offset=0.0
- joint hand_right_index_3_joint: mimic joint=hand_right_index_joint multiplier=-1.0 offset=0.0 -> joint=hand_right_index_joint multiplier=0.32 offset=0.0
- joint hand_right_middle_1_joint: mimic joint=hand_right_middle_joint multiplier=-1.0 offset=0.0 -> joint=hand_right_middle_joint multiplier=0.36 offset=0.0
- joint hand_right_middle_2_joint: mimic joint=hand_right_middle_joint multiplier=-1.0 offset=0.0 -> joint=hand_right_middle_joint multiplier=0.32 offset=0.0
- joint hand_right_middle_3_joint: mimic joint=hand_right_middle_joint multiplier=-1.0 offset=0.0 -> joint=hand_right_middle_joint multiplier=0.32 offset=0.0
